File: kicad/Daugter_boards/DB_Supply/DB_Supply_V1.sch (KiCad schematic (older format))
At the start: 28 parts, among them U1 LM555N

Commit message: creating MDL_Supply
Parts:
- added P? (x2): CONN_01X19, symbol CONN_01X19
- renumbered +3.3V1 to +3.3V, C10 to C?
Connections:
- net labels added: 03/08/2016, Supply_daugter_board
- net labels removed: -12V, -5V, 08/06/2016, 12V, 3.3V, 5V, Alimentation_Symétrique_+/-_5V;12V, GND, VCC
- wire segments 70 -> 77
- no-connect marks 18 -> 30
