File: kicad/Modules/MDL_Supply/V1.0/Supply_v1_0.sch (KiCad schematic (older format))
At the start: 28 parts, among them U1 LM555N

Commit message: adding MDL_HVC
Parts:
- U2: renamed from +12V1; value LM2940 -> LM2940CT-12
- U3: renamed from +5V1; value LM2940 -> LM2940CT-5
- U4: renamed from +3.3V1; value LM1117T -> LM1117T-3.3
- U5: renamed from -12V1; value LM2990 -> LM2990T-12
- U6: renamed from -5V1; value LM2990 -> LM2990T-5
- renumbered 2N2222 to 2N1, 2N2907 to 2N2, C6 to C10, C7 to C3, C8 to C4, C9 to C5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
Connections:
- wire segments 70 -> 45
