File: kicad/Daugter_boards/DB_TR_switch_TGC/V1/DB_TRS_TGC.sch (KiCad schematic (older format))
At the start: 3 parts, among them U1 MD0100

Commit message: update daugter boards
Parts:
- added AOP1: OPA625, symbol OPA625
- added C1: 1n, symbol C
- added P1, P10: CONN_01X19, symbol CONN_01X19
- added P2, P4, P6, P7: CONN_01X02, symbol CONN_01X02
- added P3, P5, P8, P9: SMA, symbol SMA
- added R1: 220, symbol R
Connections:
- net labels added: TGC_INH, TGC_VOUT, Transducer
- net labels removed: GND
- wire segments 2 -> 47
- no-connect marks 0 -> 4
