File: kicad/Modules/MDL_High_Voltage_Circuit/V2/MDL_HVC_V2.sch (KiCad schematic (older format))
At the start: 2 parts

Commit message: adding MLD_Pulser_V2
Parts:
- gave numbers to parts that had none: 2
Changed lines of the file:
@@
 $EndDescr
 $Comp
-L Recom U?
+L Recom U1
 U 1 1 57A30696
 P 4950 3000
-F 0 "U?" H 4950 3000 60  0000 C CNN
+F 0 "U1" H 4950 3000 60  0000 C CNN
 F 1 "Recom" H 4950 3150 60  0000 C CNN
 F 2 "" H 4650 3100 60  0000 C CNN
@@
 Connection ~ 4450 2650
 $Comp
-L GND #PWR?
+L GND #PWR01
 U 1 1 57A307B6
 P 4350 3600
-F 0 "#PWR?" H 4350 3350 50  0001 C CNN
+F 0 "#PWR01" H 4350 3350 50  0001 C CNN
 F 1 "GND" H 4350 3450 50  0000 C CNN
 F 2 "" H 4350 3600 50  0000 C CNN
@@
 Connection ~ 5450 2650
 $Comp
-L +5V #PWR?
+L +5V #PWR02
 U 1 1 57A3087B
 P 5550 2650
-F 0 "#PWR?" H 5550 2500 50  0001 C CNN
+F 0 "#PWR02" H 5550 2500 50  0001 C CNN
 F 1 "+5V" H 5550 2790 50  0000 C CNN
 F 2 "" H 5550 2650 50  0000 C CNN
@@
 $EndComp
 $Comp
-L POT RV?
+L POT RV1
 U 1 1 57A30924
 P 5600 3150
-F 0 "RV?" H 5600 3070 50  0000 C CNN
+F 0 "RV1" H 5600 3070 50  0000 C CNN
 F 1 "POT" H 5600 3150 50  0000 C CNN
 F 2 "" H 5600 3150 50  0000 C CNN

Commit message: update MDL_Pulser_V2
Parts:
- U1: value Recom -> R05-100B
Changed lines of the file:
@@
 LIBS:contrib
 LIBS:valves
-LIBS:recom
 LIBS:echopen
+LIBS:MDL_HVC_V2-cache
 EELAYER 25 0
 EELAYER END
@@
 P 4950 3000
 F 0 "U1" H 4950 3000 60  0000 C CNN
-F 1 "Recom" H 4950 3150 60  0000 C CNN
+F 1 "R05-100B" H 4950 3150 60  0000 C CNN
 F 2 "" H 4650 3100 60  0000 C CNN
 F 3 "" H 4650 3100 60  0000 C CNN
