File: kicad/Daugter_boards/DB_Envelope_detector/V1/_saved_DB_Envelope_detector_V1.sch (KiCad schematic (older format))
At the start: 5 parts, among them P1 CONN_01X19, P2 CONN_01X19

Commit message: adding mecanical repo
Parts:
- R1: footprint Resistors_ThroughHole:Resistor_Vertical_RM5mm -> Resistors_ThroughHole:Resistor_Cement_Horizontal_Meggitt-SBC-2
Changed lines of the file:
@@
 F 0 "R1" V 3430 2350 50  0000 C CNN
 F 1 "3.9k" V 3350 2350 50  0000 C CNN
-F 2 "Resistors_ThroughHole:Resistor_Vertical_RM5mm" V 3280 2350 50  0001 C CNN
+F 2 "Resistors_ThroughHole:Resistor_Cement_Horizontal_Meggitt-SBC-2" V 3280 2350 50  0001 C CNN
 F 3 "" H 3350 2350 50  0000 C CNN
 	1    3350 2350
