File: kicad/Daugter_boards/DB_Envelope_detector/V1/DB_Envelope_detector_V1.sch (KiCad schematic (older format))
At the start: 5 parts, among them P1 CONN_01X19, P2 CONN_01X19

Commit message: adding DB_Envelope_Detector
Parts:
- R1: footprint Resistors_ThroughHole:Resistor_Vertical_RM5mm -> Resistors_ThroughHole:Resistor_Cement_Horizontal_Meggitt-SBC-2
Connections:
- net GND: now reaches C1.2, P1.1 (P1), P2.1 (P1), R1.2
Changed lines of the file:
@@
 F 0 "R1" V 3430 2350 50  0000 C CNN
 F 1 "3.9k" V 3350 2350 50  0000 C CNN
-F 2 "Resistors_ThroughHole:Resistor_Vertical_RM5mm" V 3280 2350 50  0001 C CNN
+F 2 "Resistors_ThroughHole:Resistor_Cement_Horizontal_Meggitt-SBC-2" V 3280 2350 50  0001 C CNN
 F 3 "" H 3350 2350 50  0000 C CNN
 	1    3350 2350
@@
 NoConn ~ 4500 1500
 Connection ~ 3350 2200
+$Comp
+L PWR_FLAG #FLG01
+U 1 1 57AC40D5
+P 3150 3300
+F 0 "#FLG01" H 3150 3395 50  0001 C CNN
+F 1 "PWR_FLAG" H 3150 3480 50  0000 C CNN
+F 2 "" H 3150 3300 50  0000 C CNN
+F 3 "" H 3150 3300 50  0000 C CNN
+	1    3150 3300
+	1    0    0    -1
+$EndComp
+$Comp
+L GND #PWR02
+U 1 1 57AC40F8
+P 3150 3300
+F 0 "#PWR02" H 3150 3050 50  0001 C CNN
+F 1 "GND" H 3150 3150 50  0000 C CNN
+F 2 "" H 3150 3300 50  0000 C CNN
+F 3 "" H 3150 3300 50  0000 C CNN
+	1    3150 3300
+	1    0    0    -1
+$EndComp
+Connection ~ 3150 3300
 $EndSCHEMATC
