File: kicad/Daugter_boards/DB_Pulser/V1/DB_Pulser_V1.sch (KiCad schematic (older format))
At the start: 25 parts, among them P1 CONN_01X19, P2 CONN_01X02, P3 CONN_01X19, Q1 Q2N2222, Q2 Q2N2907, Q3 Q2N2222, Q4 Q2N2907, Q5 Q2N2222, Q6 Q2N2907, Q7 IRF9610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

Commit message: db pulser modif
Connections:
- net labels added: OUTPUT
Changed lines of the file:
@@
 	2450 3950 2050 3950
 NoConn ~ 2200 3950
+Text GLabel 8350 4800 2    60   Input ~ 0
+OUTPUT
 $EndSCHEMATC

Commit message: update daugter boards
Other:
- moved on the sheet: U1
Changed lines of the file:
@@
 	2450 4750 2050 4750
-Wire Wire Line
-	9850 3200 9850 5600
 Wire Wire Line
 	9850 4750 10150 4750
@@
 L SMA U1
 U 1 1 57A8AB60
-P 9300 5350
-F 0 "U1" H 9400 5450 60  0000 C CNN
-F 1 "SMA" H 9400 5550 60  0000 C CNN
-F 2 "" H 9300 5350 60  0001 C CNN
-F 3 "" H 9300 5350 60  0001 C CNN
-	1    9300 5350
+P 8750 5250
+F 0 "U1" H 8850 5350 60  0000 C CNN
+F 1 "SMA" H 8850 5450 60  0000 C CNN
+F 2 "" H 8750 5250 60  0001 C CNN
+F 3 "" H 8750 5250 60  0001 C CNN
+	1    8750 5250
 	1    0    0    -1
 $EndComp
@@
 	8000 4650 8000 5150
 Connection ~ 6500 4650
-Wire Wire Line
-	9850 5600 9050 5600
 Connection ~ 9850 4750
 Wire Wire Line
@@
 Text GLabel 8350 4800 2    60   Input ~ 0
 OUTPUT
+Wire Wire Line
+	9850 3200 9850 5450
+Wire Wire Line
+	9850 5450 8750 5450
 $EndSCHEMATC

Commit message: adding DB_Pulser
Parts:
- added C3: 33u, Capacitors_ThroughHole:C_Radial_D10_L13_P5, symbol CP
- added P4: CONN_01X02, Socket_Strips:Socket_Strip_Angled_1x02, symbol CONN_01X02
- added P5: SMA, echopen:SMA, symbol SMA
- C1, C2, C4, C5: footprint (none) -> Capacitors_ThroughHole:C_Disc_D3_P2.5
- D1, D3: footprint (none) -> Diodes_ThroughHole:Diode_DO-35_SOD27_Horizontal_RM10
- D2, D5: footprint (none) -> Connect:SMB_Straight
- P1, P3: footprint (none) -> Socket_Strips:Socket_Strip_Straight_1x19
- P2: footprint (none) -> Socket_Strips:Socket_Strip_Angled_1x02
- Q1, Q2, Q3, Q4, Q5, Q6: footprint (none) -> TO_SOT_Packages_THT:TO-18_3Pin
- Q7, Q8: footprint (none) -> TO_SOT_Packages_THT:TO-220_Neutral123_Vertical
- R1, R2, R3, R5, R6: footprint (none) -> Resistors_ThroughHole:Resistor_Horizontal_RM10mm
- U1: footprint (none) -> echopen:SMA
Connections:
- net GND: now reaches P1.1 (P1), P2.2 (P2), Q1.1 (E), Q4.3 (C), Q6.3 (C)
- net GND: now also P3.1 (P1), U1.2 (Ext), C3.1, P4.2 (P2), P5.2 (Ext)
- net at D5.1 (K), Q7.3 (S), R5.1: no longer P3.1 (P1), U1.2 (Ext)
- net at Q7.2 (D), Q8.2 (D): now also P4.1 (P1), P5.1 (In)
- net OUTPUT: no longer names the net of D2.2 (A), P2.1 (P1), Q8.3 (S), R3.2, U1.1 (In)
- net OUTPUT: now also C3.2
- no-connect marks 1 -> 35
