File: kicad/Daugter_boards/DB_Pulser/V1/_autosave-DB_Pulser_V1.kicad_pcb (KiCad board)
At the start: 2 copper layers, 43.2 x 50.8 mm, 28 parts, among them P1 CONN_01X19, P2 CONN_01X02, P3 CONN_01X19, P4 CONN_01X02, P5 SMA, Q1 Q2N2222, Q2 Q2N2907, Q3 Q2N2222, Q4 Q2N2907, Q5 Q2N2222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

Commit message: adding DB_Pulser
Routing:
- net GND: track 0.00 -> 28.3 mm
- added copper zone on B.Cu, net GND
Changed lines of the file:
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@@
   (general
     (links 57)
-    (no_connects 6)
+    (no_connects 0)
     (area 39.294999 78.664999 82.625001 129.615001)
     (thickness 1.6)
     (drawings 4)
-    (tracks 116)
+    (tracks 124)
     (zones 0)
     (modules 28)
@@
   (segment (start 57.11 109.22) (end 63.5 109.22) (width 0.25) (layer F.Cu) (net 4))
   (segment (start 63.5 109.22) (end 64.77 107.95) (width 0.25) (layer F.Cu) (net 4))
+  (segment (start 62.23 107.95) (end 62.23 101.6) (width 0.25) (layer B.Cu) (net 5))
+  (segment (start 62.23 101.6) (end 59.69 99.06) (width 0.25) (layer B.Cu) (net 5))
+  (segment (start 62.23 107.95) (end 64.77 110.49) (width 0.25) (layer B.Cu) (net 5))
+  (segment (start 69.85 115.57) (end 67.31 113.03) (width 0.25) (layer B.Cu) (net 5))
+  (segment (start 71.12 114.3) (end 69.85 115.57) (width 0.25) (layer B.Cu) (net 5))
+  (segment (start 71.12 111.76) (end 71.12 114.3) (width 0.25) (layer B.Cu) (net 5))
+  (segment (start 69.85 110.49) (end 71.12 111.76) (width 0.25) (layer B.Cu) (net 5))
+  (segment (start 64.77 110.49) (end 69.85 110.49) (width 0.25) (layer B.Cu) (net 5))
   (segment (start 73.66 125.73) (end 72.39 125.73) (width 0.25) (layer F.Cu) (net 6))
   (segment (start 66.04 123.19) (end 64.77 124.46) (width 0.25) (layer F.Cu) (net 6))
@@
     (connect_pads (clearance 0.508))
     (min_thickness 0.254)
+    (fill yes (arc_segments 16) (thermal_gap 0.508) (thermal_bridge_width 0.508))
+    (polygon
+      (pts
+        (xy 82.55 129.54) (xy 39.37 129.54) (xy 39.37 78.74) (xy 82.55 78.74)
+      )
+    )
+  )
+  (zone (net 5) (net_name GND) (layer B.Cu) (hatch edge 0.508)
+    (connect_pads (clearance 0.508))
+    (min_thickness 0.254)
