File: kicad/Daugter_boards/DB_High_Voltage/V1/DB_HV_V1.sch (KiCad schematic (older format))
At the start: 38 parts, among them P1 CONN_01X19, P2 CONN_01X02, P3 CONN_01X19, P4 SMA, Q1 QN2222, Q2 QN2222, Q3 Q2N2907, U1 LM555N

Commit message: update DB_HV, update librairy and librairy path for MDL
Parts:
- removed Q1, Q2: QN2222, TO_SOT_Packages_THT:TO-18_3Pin, symbol QN2222
- added Q1, Q2: Q2N2222, TO_SOT_Packages_THT:TO-18_3Pin, symbol Q2N2222
Connections:
- net GND: now also Q1.1 (E)
- net at P1.12 (P12), R4.1: now also Q2.3 (C)
- net at Q3.2 (B), R4.2: now also Q1.3 (C), Q2.2 (B)
- net at R3.1: now also Q1.2 (B)
- net at C3.1, Q3.1 (E): now also Q2.1 (E)
Changed lines of the file:
@@
 EESchema Schematic File Version 2
-LIBS:DB_HV_V1-rescue
 LIBS:power
 LIBS:device
@@
 LIBS:contrib
 LIBS:valves
-LIBS:echopen
 LIBS:DB_HV_V1-cache
 EELAYER 25 0
@@
 	2350 1700 2350 1500
 $Comp
-L QN2222 Q1
-U 1 1 57B37979
-P 4000 1900
-F 0 "Q1" H 4200 1975 50  0000 L CNN
-F 1 "QN2222" H 4200 1900 50  0000 L CNN
-F 2 "TO_SOT_Packages_THT:TO-18_3Pin" H 4200 1825 50  0001 L CIN
-F 3 "" H 4000 1900 50  0000 L CNN
-	1    4000 1900
-	1    0    0    -1
-$EndComp
-$Comp
-L QN2222 Q2
-U 1 1 57B37A05
-P 4900 1600
-F 0 "Q2" H 5100 1675 50  0000 L CNN
-F 1 "QN2222" H 5100 1600 50  0000 L CNN
-F 2 "TO_SOT_Packages_THT:TO-18_3Pin" H 5100 1525 50  0001 L CIN
-F 3 "" H 4900 1600 50  0000 L CNN
-	1    4900 1600
-	1    0    0    -1
-$EndComp
-$Comp
 L Q2N2907 Q3
 U 1 1 57B37A66
@@
 	1    0    0    1
 $EndComp
+$Comp
+L Q2N2222 Q1
+U 1 1 57B45C8E
+P 4000 1900
+F 0 "Q1" H 4200 1975 50  0000 L CNN
+F 1 "Q2N2222" H 4200 1900 50  0000 L CNN
+F 2 "TO_SOT_Packages_THT:TO-18_3Pin" H 4200 1825 50  0001 L CIN
+F 3 "" H 4000 1900 50  0000 L CNN
+	1    4000 1900
+	1    0    0    -1
+$EndComp
+$Comp
+L Q2N2222 Q2
+U 1 1 57B45D33
+P 4900 1600
+F 0 "Q2" H 5100 1675 50  0000 L CNN
+F 1 "Q2N2222" H 5100 1600 50  0000 L CNN
+F 2 "TO_SOT_Packages_THT:TO-18_3Pin" H 5100 1525 50  0001 L CIN
+F 3 "" H 4900 1600 50  0000 L CNN
+	1    4900 1600
+	1    0    0    -1
+$EndComp
 $EndSCHEMATC
