File: kicad/Daugter_boards/DB_Envelope_detector/V2/DB_Envelope_detector_V2.sch (KiCad schematic (older format))
At the start: 12 parts, among them P1 CONN_01X19, P2 CONN_01X19, T1 2N2222, T2 2N2907A, T3 2N2907A

Commit message: update daugter boards
Connections:
- net at P1.1 (P1), R2.2: now also P2.1 (P1)
- net +5V: no longer names the net of P2.2 (P2), R1.1, R3.1, T3.3 (E)
- net -5V: no longer names the net of C3.1, P2.18 (P18), R4.2, T2.2 (C)
Changed lines of the file:
@@
 LIBS:contrib
 LIBS:valves
+LIBS:DB_Envelope_detector_V2-cache
 EELAYER 25 0
 EELAYER END
@@
 	6750 4400 6750 4350
 Connection ~ 6750 4350
-Text Label 7200 4800 0    60   ~ 0
--5V
-Text Label 7200 3150 0    60   ~ 0
-+5V
 Wire Wire Line
 	5700 4800 7450 4800
@@
 	7550 4550 7550 4350
 Wire Wire Line
-	5250 4950 3650 4950
+	3650 4950 8300 4950
 Wire Wire Line
 	8300 4850 7750 4850
@@
 NoConn ~ 7750 4550
 NoConn ~ 7450 4350
+Connection ~ 5250 4950
 $EndSCHEMATC

Commit message: adding DB_Envelope_Detector
Parts:
- C1, C2, C3: footprint (none) -> Capacitors_ThroughHole:C_Disc_D6_P5
- P1, P2: footprint (none) -> Socket_Strips:Socket_Strip_Straight_1x19
- R1, R2, R3, R4: footprint (none) -> Resistors_ThroughHole:Resistor_Ceramic_Horizontal_L19mm-W8mm-H8mm-p25mm
- T1, T2, T3: footprint (none) -> Transistors_OldSowjetAera:OldSowjetaera_Transistor_Type-II_BigPads
Connections:
- net at R1.2, R2.1: now also C1.1, T1.1 (B)
- net GND: now reaches P1.1 (P1), P2.1 (P1), R2.2
- no-connect marks 3 -> 35
Changed lines of the file:
@@
 F 0 "R1" V 5330 3400 50  0000 C CNN
 F 1 "2800" V 5250 3400 50  0000 C CNN
-F 2 "" V 5180 3400 50  0000 C CNN
+F 2 "Resistors_ThroughHole:Resistor_Ceramic_Horizontal_L19mm-W8mm-H8mm-p25mm" V 5180 3400 50  0001 C CNN
 F 3 "" H 5250 3400 50  0000 C CNN
 	1    5250 3400
@@
 F 0 "C1" H 4825 3950 50  0000 L CNN
 F 1 "10nF" H 4825 3750 50  0000 L CNN
-F 2 "" H 4838 3700 50  0000 C CNN
+F 2 "Capacitors_ThroughHole:C_Disc_D6_P5" H 4838 3700 50  0001 C CNN
 F 3 "" H 4800 3850 50  0000 C CNN
 	1    4800 3850
@@
 F 0 "R2" V 5330 4300 50  0000 C CNN
 F 1 "1000" V 5250 4300 50  0000 C CNN
-F 2 "" V 5180 4300 50  0000 C CNN
+F 2 "Resistors_ThroughHole:Resistor_Ceramic_Horizontal_L19mm-W8mm-H8mm-p25mm" V 5180 4300 50  0001 C CNN
 F 3 "" H 5250 4300 50  0000 C CNN
 	1    5250 4300
@@
 F 0 "R3" V 5780 3400 50  0000 C CNN
 F 1 "330" V 5700 3400 50  0000 C CNN
-F 2 "" V 5630 3400 50  0000 C CNN
+F 2 "Resistors_ThroughHole:Resistor_Ceramic_Horizontal_L19mm-W8mm-H8mm-p25mm" V 5630 3400 50  0001 C CNN
 F 3 "" H 5700 3400 50  0000 C CNN
 	1    5700 3400
@@
 F 0 "T1" H 5850 3950 50  0000 R CNN
 F 1 "2N2222" H 5900 3800 50  0000 R BNN
-F 2 "" H 5800 3950 50  0000 C CNN
+F 2 "Transistors_OldSowjetAera:OldSowjetaera_Transistor_Type-II_BigPads" H 5800 3950 50  0001 C CNN
 F 3 "" H 5600 3850 50  0000 C CNN
 	1    5600 3850
@@
 F 0 "T2" H 5750 4450 50  0000 C CNN
 F 1 "2N2907A" H 5650 4150 50  0000 C CNN
-F 2 "" H 6000 4400 50  0000 C CNN
+F 2 "Transistors_OldSowjetAera:OldSowjetaera_Transistor_Type-II_BigPads" H 6000 4400 50  0001 C CNN
 F 3 "" H 5800 4300 50  0000 C CNN
 	1    5800 4300
@@
 F 0 "R4" V 6430 4550 50  0000 C CNN
 F 1 "330" V 6350 4550 50  0000 C CNN
-F 2 "" V 6280 4550 50  0000 C CNN
+F 2 "Resistors_ThroughHole:Resistor_Ceramic_Horizontal_L19mm-W8mm-H8mm-p25mm" V 6280 4550 50  0001 C CNN
 F 3 "" H 6350 4550 50  0000 C CNN
 	1    6350 4550
@@
 F 0 "T3" H 6200 3750 50  0000 C CNN
 F 1 "2N2907A" H 6100 3450 50  0000 C CNN
-F 2 "" H 6450 3700 50  0000 C CNN
+F 2 "Transistors_OldSowjetAera:OldSowjetaera_Transistor_Type-II_BigPads" H 6450 3700 50  0001 C CNN
 F 3 "" H 6250 3600 50  0000 C CNN
 	1    6250 3600
@@
 Wire Wire Line
 	6350 4300 6350 4250
-Connection ~ 6350 4250
 Wire Wire Line
 	5700 4500 5700 4800
@@
 F 0 "C2" H 6125 3950 50  0000 L CNN
 F 1 "1nF" H 6125 3750 50  0000 L CNN
-F 2 "" H 6138 3700 50  0000 C CNN
+F 2 "Capacitors_ThroughHole:C_Disc_D6_P5" H 6138 3700 50  0001 C CNN
 F 3 "" H 6100 3850 50  0000 C CNN
 	1    6100 3850
@@
 F 0 "C3" H 6775 4650 50  0000 L CNN
 F 1 "33nF" H 6775 4450 50  0000 L CNN
-F 2 "" H 6788 4400 50  0000 C CNN
+F 2 "Capacitors_ThroughHole:C_Disc_D6_P5" H 6788 4400 50  0001 C CNN
 F 3 "" H 6750 4550 50  0000 C CNN
 	1    6750 4550
@@
 F 0 "P1" H 3450 5050 50  0000 C CNN
 F 1 "CONN_01X19" V 3550 4050 50  0000 C CNN
-F 2 "" H 3450 4050 50  0000 C CNN
+F 2 "Socket_Strips:Socket_Strip_Straight_1x19" H 3450 4050 50  0001 C CNN
 F 3 "" H 3450 4050 50  0000 C CNN
 	1    3450 4050
@@
 F 0 "P2" H 8500 5050 50  0000 C CNN
 F 1 "CONN_01X19" V 8600 4050 50  0000 C CNN
-F 2 "" H 8500 4050 50  0000 C CNN
+F 2 "Socket_Strips:Socket_Strip_Straight_1x19" H 8500 4050 50  0001 C CNN
 F 3 "" H 8500 4050 50  0000 C CNN
 	1    8500 4050
@@
 NoConn ~ 7450 4350
 Connection ~ 5250 4950
+$Comp
+L PWR_FLAG #FLG01
+U 1 1 57AC81D8
+P 4600 4950
+F 0 "#FLG01" H 4600 5045 50  0001 C CNN
+F 1 "PWR_FLAG" H 4600 5130 50  0000 C CNN
+F 2 "" H 4600 4950 50  0000 C CNN
+F 3 "" H 4600 4950 50  0000 C CNN
+	1    4600 4950
+	1    0    0    -1
+$EndComp
+$Comp
+L GND #PWR02
+U 1 1 57AC8210
+P 4600 4950
+F 0 "#PWR02" H 4600 4700 50  0001 C CNN
+F 1 "GND" H 4600 4800 50  0000 C CNN
+F 2 "" H 4600 4950 50  0000 C CNN
+F 3 "" H 4600 4950 50  0000 C CNN
+	1    4600 4950
+	1    0    0    -1
+$EndComp
+Connection ~ 4600 4950
+NoConn ~ 3650 3150
+NoConn ~ 3650 3250
+NoConn ~ 3650 3350
+NoConn ~ 3650 3450
+NoConn ~ 3650 3550
+NoConn ~ 3650 3650
+NoConn ~ 3650 3750
+NoConn ~ 3650 3850
+NoConn ~ 3650 4050
+NoConn ~ 3650 4150
+NoConn ~ 3650 4250
+NoConn ~ 3650 4350
+NoConn ~ 3650 4450
+NoConn ~ 3650 4550
+NoConn ~ 3650 4750
+NoConn ~ 3650 4850
+NoConn ~ 8300 3150
+NoConn ~ 8300 3350
+NoConn ~ 8300 3450
+NoConn ~ 8300 3550
+NoConn ~ 8300 3650
+NoConn ~ 8300 3750
+NoConn ~ 8300 3850
+NoConn ~ 8300 3950
+NoConn ~ 8300 4050
+NoConn ~ 8300 4150
+NoConn ~ 8300 4250
+NoConn ~ 8300 4350
+NoConn ~ 8300 4450
+NoConn ~ 8300 4650
+NoConn ~ 8300 4750
+Connection ~ 5250 3850
+Connection ~ 6350 4250
+Connection ~ 6350 4300
+NoConn ~ 3650 3950
 $EndSCHEMATC

Commit message: update DB_Envelope_Detector with correct librairy and footprint
Parts:
- removed T1: 2N2222, Transistors_OldSowjetAera:OldSowjetaera_Transistor_Type-II_BigPads, symbol Q_NPN_BCE
- removed T2, T3: 2N2907A, Transistors_OldSowjetAera:OldSowjetaera_Transistor_Type-II_BigPads, symbol Q_PNP_BCE
- added Q1: Q2N2222, TO_SOT_Packages_THT:TO-18_3Pin, symbol Q2N2222
- added Q2, Q3: Q2N2907, TO_SOT_Packages_THT:TO-18_3Pin, symbol Q2N2907
Connections:
- net at P2.2 (P2), R1.1, R3.1: now also Q3.1 (E)
- net at C1.1, R1.2, R2.1: now also Q1.2 (B)
- net at C2.2, R3.2: now also Q1.3 (C), Q3.2 (B)
- net at C2.1, C3.2, P2.5 (P5)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: now also Q2.2 (B), Q3.3 (C)
- net at C3.1, P2.18 (P18), R4.2: now also Q2.3 (C)
- new net: Q1.1 (E), Q2.1 (E)
Changed lines of the file:
@@
 LIBS:contrib
 LIBS:valves
+LIBS:echopen
 LIBS:DB_Envelope_detector_V2-cache
 EELAYER 25 0
@@
 	1    0    0    -1
 $EndComp
-$Comp
-L Q_NPN_BCE T1
-U 1 1 576BE9ED
-P 5600 3850
-F 0 "T1" H 5850 3950 50  0000 R CNN
-F 1 "2N2222" H 5900 3800 50  0000 R BNN
-F 2 "Transistors_OldSowjetAera:OldSowjetaera_Transistor_Type-II_BigPads" H 5800 3950 50  0001 C CNN
-F 3 "" H 5600 3850 50  0000 C CNN
-	1    5600 3850
-	1    0    0    -1
-$EndComp
 Wire Wire Line
 	5250 3550 5250 4150
 Wire Wire Line
-	5400 3850 4950 3850
-$Comp
-L Q_PNP_BCE T2
-U 1 1 576BEED3
-P 5800 4300
-F 0 "T2" H 5750 4450 50  0000 C CNN
-F 1 "2N2907A" H 5650 4150 50  0000 C CNN
-F 2 "Transistors_OldSowjetAera:OldSowjetaera_Transistor_Type-II_BigPads" H 6000 4400 50  0001 C CNN
-F 3 "" H 5800 4300 50  0000 C CNN
-	1    5800 4300
-	-1   0    0    1
-$EndComp
+	4950 3850 5400 3850
 $Comp
 L R R4
@@
 	1    0    0    -1
 $EndComp
-$Comp
-L Q_PNP_BCE T3
-U 1 1 576C07B0
-P 6250 3600
-F 0 "T3" H 6200 3750 50  0000 C CNN
-F 1 "2N2907A" H 6100 3450 50  0000 C CNN
-F 2 "Transistors_OldSowjetAera:OldSowjetaera_Transistor_Type-II_BigPads" H 6450 3700 50  0001 C CNN
-F 3 "" H 6250 3600 50  0000 C CNN
-	1    6250 3600
-	1    0    0    1
-$EndComp
 Wire Wire Line
 	5250 3250 5250 3150
@@
 Connection ~ 5700 3150
 Wire Wire Line
-	5700 3650 5700 3550
-Wire Wire Line
-	6050 3600 5700 3600
+	5700 3550 5700 3650
+Wire Wire Line
+	5700 3600 6050 3600
 Connection ~ 5700 3600
 Wire Wire Line
@@
 Connection ~ 6350 3850
 Wire Wire Line
-	6350 3400 6350 3150
+	6350 3150 6350 3400
 Connection ~ 6350 3150
 Wire Wire Line
@@
 $EndComp
 Wire Wire Line
-	6750 4700 6750 4800
+	6750 4800 6750 4700
 Connection ~ 6750 4800
 Wire Wire Line
@@
 	5700 4800 7450 4800
 Wire Wire Line
-	5250 4450 5250 4950
+	5250 4950 5250 4450
 Text Label 7450 7500 0    60   ~ 12
 Detection_d'enveloppe
@@
 Connection ~ 6350 4300
 NoConn ~ 3650 3950
+$Comp
+L Q2N2222 Q1
+U 1 1 57B43F1F
+P 5600 3850
+F 0 "Q1" H 5800 3925 50  0000 L CNN
+F 1 "Q2N2222" H 5800 3850 50  0000 L CNN
+F 2 "TO_SOT_Packages_THT:TO-18_3Pin" H 5800 3775 50  0001 L CIN
+F 3 "" H 5600 3850 50  0000 L CNN
+	1    5600 3850
+	1    0    0    -1
+$EndComp
+$Comp
+L Q2N2907 Q2
+U 1 1 57B43F5E
+P 5800 4300
+F 0 "Q2" H 6000 4375 50  0000 L CNN
+F 1 "Q2N2907" H 6000 4300 50  0000 L CNN
+F 2 "TO_SOT_Packages_THT:TO-18_3Pin" H 6100 4150 50  0001 L CIN
+F 3 "" H 5800 4300 50  0000 L CNN
+	1    5800 4300
+	-1   0    0    1
+$EndComp
+$Comp
+L Q2N2907 Q3
+U 1 1 57B4408A
+P 6250 3600
+F 0 "Q3" H 6450 3675 50  0000 L CNN
+F 1 "Q2N2907" H 6450 3600 50  0000 L CNN
+F 2 "TO_SOT_Packages_THT:TO-18_3Pin" H 6550 3450 50  0001 L CIN
+F 3 "" H 6250 3600 50  0000 L CNN
+	1    6250 3600
+	1    0    0    1
+$EndComp
 $EndSCHEMATC

Commit message: update librairy with correct nomenclature of transistor
Parts:
- removed Q1: Q2N2222, TO_SOT_Packages_THT:TO-18_3Pin, symbol Q2N2222
- removed Q2, Q3: Q2N2907, TO_SOT_Packages_THT:TO-18_3Pin, symbol Q2N2907
- added Q1: 2N2222, TO_SOT_Packages_THT:TO-18_3Pin, symbol 2N2222
- added Q2, Q3: 2N2907, TO_SOT_Packages_THT:TO-18_3Pin, symbol 2N2907
Connections:
- net at P2.2 (P2), R1.1, R3.1: now also Q3.1 (E)
- net at C1.1, R1.2, R2.1: now also Q1.2 (B)
- net at C2.2, R3.2: now also Q1.3 (C), Q3.2 (B)
- net at C2.1, C3.2, P2.5 (P5)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: now also Q2.2 (B), Q3.3 (C)
- net at C3.1, P2.18 (P18), R4.2: now also Q2.3 (C)
- new net: Q1.1 (E), Q2.1 (E)
Changed lines of the file:
@@
 NoConn ~ 3650 3950
 $Comp
-L Q2N2222 Q1
-U 1 1 57B43F1F
+L 2N2222 Q1
+U 1 1 57B448C8
 P 5600 3850
 F 0 "Q1" H 5800 3925 50  0000 L CNN
-F 1 "Q2N2222" H 5800 3850 50  0000 L CNN
+F 1 "2N2222" H 5800 3850 50  0000 L CNN
 F 2 "TO_SOT_Packages_THT:TO-18_3Pin" H 5800 3775 50  0001 L CIN
 F 3 "" H 5600 3850 50  0000 L CNN
@@
 $EndComp
 $Comp
-L Q2N2907 Q2
-U 1 1 57B43F5E
+L 2N2907 Q2
+U 1 1 57B44946
 P 5800 4300
 F 0 "Q2" H 6000 4375 50  0000 L CNN
-F 1 "Q2N2907" H 6000 4300 50  0000 L CNN
+F 1 "2N2907" H 6000 4300 50  0000 L CNN
 F 2 "TO_SOT_Packages_THT:TO-18_3Pin" H 6100 4150 50  0001 L CIN
 F 3 "" H 5800 4300 50  0000 L CNN
@@
 $EndComp
 $Comp
-L Q2N2907 Q3
-U 1 1 57B4408A
+L 2N2907 Q3
+U 1 1 57B44A85
 P 6250 3600
 F 0 "Q3" H 6450 3675 50  0000 L CNN
-F 1 "Q2N2907" H 6450 3600 50  0000 L CNN
+F 1 "2N2907" H 6450 3600 50  0000 L CNN
 F 2 "TO_SOT_Packages_THT:TO-18_3Pin" H 6550 3450 50  0001 L CIN
 F 3 "" H 6250 3600 50  0000 L CNN
