File: kicad/Modules/MDL_High_Voltage_Circuit/V1/MDL_HVC_V1.sch (KiCad schematic (older format))
At the start: 34 parts, among them U1 LM555N

Commit message: update DB_HV, update librairy and librairy path for MDL
Parts:
- removed 2N1, 2N2222_1: Q_NPN_BCE, symbol Q_NPN_BCE
- removed 2N2: Q_PNP_BCE, symbol Q_PNP_BCE
- added Q1, Q2: Q2N2222, symbol Q2N2222
- added Q3: Q2N2907, symbol Q2N2907
Connections:
- net GND: now also Q1.1 (E), Q3.3 (C)
- net VCC: now also Q2.3 (C)
- net at R3.1: now also Q1.2 (B)
- net at R4.2: now also Q1.3 (C), Q2.2 (B), Q3.2 (B)
- net at C3.1: now also Q2.1 (E), Q3.1 (E)
Changed lines of the file:
@@
 LIBS:contrib
 LIBS:valves
+LIBS:echopen
 LIBS:MDL_HVC_V1-cache
 EELAYER 25 0
@@
 $EndComp
 $Comp
-L Q_PNP_BCE 2N2
-U 1 1 57A21CAB
-P 5150 2050
-F 0 "2N2" H 5450 2100 50  0000 R CNN
-F 1 "Q_PNP_BCE" H 5750 2000 50  0000 R CNN
-F 2 "" H 5350 2150 50  0001 C CNN
-F 3 "" H 5150 2050 50  0000 C CNN
-	1    5150 2050
-	1    0    0    1
-$EndComp
-$Comp
-L Q_NPN_BCE 2N2222_1
-U 1 1 57A21CAA
-P 5150 1650
-F 0 "2N2222_1" H 5450 1700 50  0000 R CNN
-F 1 "Q_NPN_BCE" H 5750 1600 50  0000 R CNN
-F 2 "" H 5350 1750 50  0001 C CNN
-F 3 "" H 5150 1650 50  0000 C CNN
-	1    5150 1650
-	1    0    0    -1
-$EndComp
-$Comp
 L R R4
 U 1 1 57A21CA9
@@
 F 3 "" H 4350 1600 50  0000 C CNN
 	1    4350 1600
-	1    0    0    -1
-$EndComp
-$Comp
-L Q_NPN_BCE 2N1
-U 1 1 57A21CA8
-P 4250 1950
-F 0 "2N1" H 4550 2000 50  0000 R CNN
-F 1 "Q_NPN_BCE" H 4850 1900 50  0000 R CNN
-F 2 "" H 4450 2050 50  0001 C CNN
-F 3 "" H 4250 1950 50  0000 C CNN
-	1    4250 1950
 	1    0    0    -1
 $EndComp
@@
 Wire Wire Line
 	10900 2900 10900 3100
+$Comp
+L Q2N2222 Q1
+U 1 1 57B42EE7
+P 4250 1950
+F 0 "Q1" H 4450 2025 50  0000 L CNN
+F 1 "Q2N2222" H 4450 1950 50  0000 L CNN
+F 2 "" H 4450 1875 50  0000 L CIN
+F 3 "" H 4250 1950 50  0000 L CNN
+	1    4250 1950
+	1    0    0    -1
+$EndComp
+$Comp
+L Q2N2222 Q2
+U 1 1 57B42F68
+P 5150 1650
+F 0 "Q2" H 5350 1725 50  0000 L CNN
+F 1 "Q2N2222" H 5350 1650 50  0000 L CNN
+F 2 "" H 5350 1575 50  0000 L CIN
+F 3 "" H 5150 1650 50  0000 L CNN
+	1    5150 1650
+	1    0    0    -1
+$EndComp
+$Comp
+L Q2N2907 Q3
+U 1 1 57B42FF3
+P 5150 2050
+F 0 "Q3" H 5350 2125 50  0000 L CNN
+F 1 "Q2N2907" H 5350 2050 50  0000 L CNN
+F 2 "" H 5450 1900 50  0000 L CIN
+F 3 "" H 5150 2050 50  0000 L CNN
+	1    5150 2050
+	1    0    0    1
+$EndComp
 $EndSCHEMATC

Commit message: update figures and nomenclature of MDLs
Parts:
- D1, D12: value 400x -> 1N4001
Changed lines of the file:
@@
 P 6300 2000
 F 0 "D1" H 6300 2100 50  0000 C CNN
-F 1 "400x" H 6300 1900 50  0000 C CNN
+F 1 "1N4001" H 6300 1900 50  0000 C CNN
 F 2 "" H 6300 2000 50  0000 C CNN
 F 3 "" H 6300 2000 50  0000 C CNN
@@
 P 10900 2750
 F 0 "D12" H 10900 2850 50  0000 C CNN
-F 1 "400x" H 10900 2650 50  0000 C CNN
+F 1 "1N4001" H 10900 2650 50  0000 C CNN
 F 2 "" H 10900 2750 50  0000 C CNN
 F 3 "" H 10900 2750 50  0000 C CNN

Commit message: update MDLs with new librairy
Parts:
- removed Q1, Q2: Q2N2222, symbol Q2N2222
- removed Q3: Q2N2907, symbol Q2N2907
- added Q1, Q2: 2N2222, symbol 2N2222
- added Q3: 2N2907, symbol 2N2907
Connections:
- net GND: now also Q1.1 (E), Q3.3 (C)
- net VCC: now also Q2.3 (C)
- net at R4.2: now also Q1.3 (C), Q2.2 (B), Q3.2 (B)
- net at R3.1: now also Q1.2 (B)
- net at C3.1: now also Q2.1 (E), Q3.1 (E)
Changed lines of the file:
@@
 	10900 2900 10900 3100
 $Comp
-L Q2N2222 Q1
-U 1 1 57B42EE7
+L 2N2222 Q1
+U 1 1 57B46F76
 P 4250 1950
 F 0 "Q1" H 4450 2025 50  0000 L CNN
-F 1 "Q2N2222" H 4450 1950 50  0000 L CNN
+F 1 "2N2222" H 4450 1950 50  0000 L CNN
 F 2 "" H 4450 1875 50  0000 L CIN
 F 3 "" H 4250 1950 50  0000 L CNN
@@
 $EndComp
 $Comp
-L Q2N2222 Q2
-U 1 1 57B42F68
+L 2N2222 Q2
+U 1 1 57B47024
 P 5150 1650
 F 0 "Q2" H 5350 1725 50  0000 L CNN
-F 1 "Q2N2222" H 5350 1650 50  0000 L CNN
+F 1 "2N2222" H 5350 1650 50  0000 L CNN
 F 2 "" H 5350 1575 50  0000 L CIN
 F 3 "" H 5150 1650 50  0000 L CNN
@@
 $EndComp
 $Comp
-L Q2N2907 Q3
-U 1 1 57B42FF3
+L 2N2907 Q3
+U 1 1 57B470CA
 P 5150 2050
 F 0 "Q3" H 5350 2125 50  0000 L CNN
-F 1 "Q2N2907" H 5350 2050 50  0000 L CNN
+F 1 "2N2907" H 5350 2050 50  0000 L CNN
 F 2 "" H 5450 1900 50  0000 L CIN
 F 3 "" H 5150 2050 50  0000 L CNN
