File: kicad/Daugter_boards/DB_Link/DB_Link.kicad_pcb (KiCad board)
At the start: 2 copper layers, 45.7 x 50.8 mm, 2 parts, among them P1 CONN_01X19, P2 CONN_01X19

Commit message: improve DB_Mother_Board finish
Other:
- board text added: "+12V"
- board text added: "+18V"
- board text added: "+3.3V"
- board text added: "+5V"
- board text added: "-12V"
- board text added: "-5V"
- board text added: "B1"
- board text added: "B2"
- board text added: "Encoder"
- board text added: "Envelope"
- board text added: "Filtered TGC"
- board text added: "GND"
- board text added: "Motor PWM"
- board text added: "Ramp"
- board text added: "TGC OUT"
- board text added: "Tir OFF"
- board text added: "Tir ON"
- board text added: "Top Tour"
- board text added: "Trigger RP"
Changed lines of the file:
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@@
     (links 19)
     (no_connects 0)
-    (area 105.334999 100.376666 154.765 153.745001)
+    (area 105.334999 102.794999 151.205001 153.745001)
     (thickness 1.6)
-    (drawings 4)
+    (drawings 23)
     (tracks 19)
     (zones 0)
@@
     (pad_to_mask_clearance 0.2)
     (aux_axis_origin 0 0)
-    (visible_elements FFFFFF7F)
+    (visible_elements 7FFFFFFF)
     (pcbplotparams
       (layerselection 0x00030_80000001)
@@
     (descr "Through hole socket strip")
     (tags "socket strip")
-    (fp_text reference P1 (at 0 -5.1 270) (layer F.SilkS)
+    (fp_text reference P1 (at 0 -3.175 270) (layer F.SilkS)
       (effects (font (size 1 1) (thickness 0.15)))
     )
@@
     (descr "Through hole socket strip")
     (tags "socket strip")
-    (fp_text reference P2 (at 0 -5.1 270) (layer F.SilkS)
+    (fp_text reference P2 (at 0 2.54 270) (layer F.SilkS)
       (effects (font (size 1 1) (thickness 0.15)))
     )
@@
     )
   )
+  (gr_text +3.3V (at 146.685 151.13) (layer B.Cu)
+    (effects (font (size 1.5 1.5) (thickness 0.3)) (justify left mirror))
+  )
+  (gr_text -5V (at 146.685 148.59) (layer B.Cu)
+    (effects (font (size 1.5 1.5) (thickness 0.3)) (justify left mirror))
+  )
+  (gr_text B2 (at 145.415 146.05) (layer B.Cu)
+    (effects (font (size 1.5 1.5) (thickness 0.3)) (justify mirror))
+  )
+  (gr_text B1 (at 146.685 143.51) (layer B.Cu)
+    (effects (font (size 1.5 1.5) (thickness 0.3)) (justify left mirror))
+  )
+  (gr_text Encoder (at 146.685 140.97) (layer B.Cu)
+    (effects (font (size 1.5 1.5) (thickness 0.3)) (justify left mirror))
+  )
+  (gr_text "Motor PWM" (at 146.685 138.43) (layer B.Cu)
+    (effects (font (size 1.5 1.5) (thickness 0.3)) (justify left mirror))
+  )
+  (gr_text "Top Tour" (at 146.685 135.89) (layer B.Cu)
+    (effects (font (size 1.5 1.5) (thickness 0.3)) (justify left mirror))
+  )
+  (gr_text +18V (at 146.685 133.35) (layer B.Cu)
+    (effects (font (size 1.5 1.5) (thickness 0.3)) (justify left mirror))
+  )
+  (gr_text "Trigger RP" (at 146.685 130.81) (layer B.Cu)
+    (effects (font (size 1.5 1.5) (thickness 0.3)) (justify left mirror))
+  )
+  (gr_text "Tir OFF" (at 146.685 128.27) (layer B.Cu)
+    (effects (font (size 1.5 1.5) (thickness 0.3)) (justify left mirror))
+  )
+  (gr_text "Tir ON" (at 146.685 125.73) (layer B.Cu)
+    (effects (font (size 1.5 1.5) (thickness 0.3)) (justify left mirror))
+  )
+  (gr_text -12V (at 146.685 123.19) (layer B.Cu)
+    (effects (font (size 1.5 1.5) (thickness 0.3)) (justify left mirror))
+  )
+  (gr_text Ramp (at 146.685 120.65) (layer B.Cu)
+    (effects (font (size 1.5 1.5) (thickness 0.3)) (justify left mirror))
+  )
+  (gr_text "+12V\n" (at 146.685 118.11) (layer B.Cu)
+    (effects (font (size 1.5 1.5) (thickness 0.3)) (justify left mirror))
+  )
+  (gr_text Envelope (at 146.685 115.57) (layer B.Cu)
+    (effects (font (size 1.5 1.5) (thickness 0.3)) (justify left mirror))
+  )
+  (gr_text "Filtered TGC" (at 146.685 113.03) (layer B.Cu)
+    (effects (font (size 1.5 1.5) (thickness 0.3)) (justify left mirror))
+  )
+  (gr_text "TGC OUT" (at 146.685 110.49) (layer B.Cu)
+    (effects (font (size 1.5 1.5) (thickness 0.3)) (justify left mirror))
+  )
+  (gr_text +5V (at 146.685 107.95) (layer B.Cu)
+    (effects (font (size 1.5 1.5) (thickness 0.3)) (justify left mirror))
+  )
+  (gr_text GND (at 146.685 105.41) (layer B.Cu)
+    (effects (font (size 1.5 1.5) (thickness 0.3)) (justify left mirror))
+  )
   (gr_line (start 151.13 102.87) (end 105.41 102.87) (angle 90) (layer Edge.Cuts) (width 0.15))
